Commit message: updated urdf file to get rid of non-uniform axes; added exercise 1,2 readmes

File: iCub/full.urdf (robot description, URDF)
Before this commit: robot iCub, 103 links, 102 joints
Joints:
- joint l_shoulder_pitch: axis 0.965926 0.0 0.258819 -> 0.9659258492011169 0 0.25881895959357540
- joint l_shoulder_roll: axis -0.258819 2.77555756156e-17 0.965926 -> -0.2588189595935754 0 0.9659258492011169
- joint l_shoulder_yaw: axis 0.965925843882 2.22044604925e-16 0.258818979447 -> 0.9659258492011169 0 0.2588189595935754
- joint l_wrist_pitch: axis 0.258818979447 0.0 -0.965925843882 -> 0.2588189595935754 0.0 -0.9659258492011169
- joint l_wrist_prosup: axis 0.965925843882 2.22044604925e-16 0.258818979447 -> 0.9659258492011169 0 0.2588189595935754
- joint r_shoulder_pitch: axis -0.965925926173 0.0 0.258819275525 -> -0.9659257753743923 0.0 0.25881923511860305
- joint r_shoulder_roll: axis -0.258819 -2.77555756156e-17 -0.965926 -> -0.2588189595935754 0 -0.9659258492011169
- joint r_shoulder_yaw: axis 0.965925843882 -2.22044604925e-16 -0.258818979447 -> 0.9659258492011169 0 -0.2588189595935754
- joint r_wrist_pitch: axis 0.258818979447 0.0 0.965925843882 -> 0.25881895959357540 0 0.9659258492011169
- joint r_wrist_prosup: axis 0.965925843882 -2.22044604925e-16 -0.258818979447 -> 0.9659258492011169 0 -0.2588189595935754

File: iCub/full_vhacd.urdf (robot description, URDF)
Before this commit: robot iCub, 103 links, 102 joints
Joints:
- joint l_shoulder_pitch: axis 0.965926 0.0 0.258819 -> 0.9659258492011169 0.0 0.2588189595935754
- joint l_shoulder_roll: axis -0.258819 2.77555756156e-17 0.965926 -> -0.2588189595935754 0.0 0.9659258492011169
- joint l_shoulder_yaw: axis 0.965925843882 2.22044604925e-16 0.258818979447 -> 0.9659258492011169 0.0 0.2588189595935754
- joint l_wrist_pitch: axis 0.258818979447 0.0 -0.965925843882 -> 0.2588189595935754 0.0 -0.9659258492011169
- joint l_wrist_prosup: axis 0.965925843882 2.22044604925e-16 0.258818979447 -> 0.9659258492011169 0.0 0.2588189595935754
- joint r_shoulder_pitch: axis -0.965925926173 0.0 0.258819275525 -> -0.9659257753743923 0.0 0.25881923511860305
- joint r_shoulder_roll: axis -0.258819 -2.77555756156e-17 -0.965926 -> -0.2588189595935754 0.0 -0.9659258492011169
- joint r_shoulder_yaw: axis 0.965925843882 -2.22044604925e-16 -0.258818979447 -> 0.9659258492011169 0.0 -0.2588189595935754
- joint r_wrist_pitch: axis 0.258818979447 0.0 0.965925843882 -> 0.2588189595935754 0.0 0.9659258492011169
- joint r_wrist_prosup: axis 0.965925843882 -2.22044604925e-16 -0.258818979447 -> 0.9659258492011169 0.0 -0.2588189595935754

Commit message: Bugfixes added check fo -1 in in raybatch which means no contact; added correct collision mesh for icub sole/foot/boot

File: iCub/full.urdf (robot description, URDF)
Before this commit: robot iCub, 103 links, 102 joints
Links:
- link l_foot: geometry collision mesh filename=package://iCub/meshes/visual/sim_sea_2-5_l_sole_prt-binary.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 scale=0.001 0.001 0.001; visual mesh filename=package://iCub/meshes/visual/sim_sea_2-5_l_sole_prt-binary.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 scale=0.001 0.001 0.001
- link r_foot: geometry collision mesh filename=package://iCub/meshes/visual/sim_sea_2-5_r_sole_prt-binary.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 scale=0.001 0.001 0.001; visual mesh filename=package://iCub/meshes/visual/sim_sea_2-5_r_sole_prt-binary.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 scale=0.001 0.001 0.001

File: iCub/full_vhacd.urdf (robot description, URDF)
Before this commit: robot iCub, 103 links, 102 joints
Links:
- link l_foot: geometry collision mesh filename=package://iCub/meshes/vhacd/sim_sea_2-5_l_sole_prt-binary_v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 scale=0.001 0.001 0.001; visual mesh filename=package://iCub/meshes/visual/sim_sea_2-5_l_sole_prt-binary.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 scale=0.001 0.001 0.001
- link r_foot: geometry collision mesh filename=package://iCub/meshes/vhacd/sim_sea_2-5_r_sole_prt-binary_v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 scale=0.001 0.001 0.001; visual mesh filename=package://iCub/meshes/visual/sim_sea_2-5_r_sole_prt-binary.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 scale=0.001 0.001 0.001

Commit message: Changes for grasper added timeout to movements; changed behaviour when joints outside limits are inserted; visualizer now correctly shows when fixed objects change their position

File: iCub/full.urdf (robot description, URDF)
Before this commit: robot iCub, 103 links, 102 joints
Links:
- link l_eye_pupil: geometry collision mesh filename=package://iCub/meshes/visual/l_eye_pupil.obj scale=1.0 1.0 1.0; visual mesh filename=package://iCub/meshes/visual/l_eye_pupil.obj scale=1.0 1.0 1.0
- link r_eye_pupil: geometry collision mesh filename=package://iCub/meshes/visual/r_eye_pupil.obj scale=1.0 1.0 1.0; visual mesh filename=package://iCub/meshes/visual/r_eye_pupil.obj scale=1.0 1.0 1.0

File: iCub/full_vhacd.urdf (robot description, URDF)
Before this commit: robot iCub, 103 links, 102 joints
Links:
- link l_eye_pupil: geometry collision mesh filename=package://iCub/meshes/vhacd/l_eye_pupil_vhacd.obj scale=1.0 1.0 1.0; visual mesh filename=package://iCub/meshes/visual/l_eye_pupil.obj scale=1.0 1.0 1.0
- link r_eye_pupil: geometry collision mesh filename=package://iCub/meshes/vhacd/r_eye_pupil_vhacd.obj scale=1.0 1.0 1.0; visual mesh filename=package://iCub/meshes/visual/r_eye_pupil.obj scale=1.0 1.0 1.0

Commit message: Merge from dev (#5)
* icub_pybullet/examples/

* Updates towards v1.0
changed time management in update_simulation()
removed try/except in imports in examples
added option for web visualizer through configs

* Workflow start
added action to build and push image to dockerhub
added gitpod dockerfile
added .gitpod.yml

* Updated vnc and gitpod dockers

* Fixed error in Dockerfile.gitpod

* Fixed error in Dockerfile.gitpod

* Updated workflow; updated standard Dockerfile

* Updated numpy version

* Updated Pycharm.desktop file

* Changed to numpy lower than 2

* Auto workflow

* Added multiplatform build

* vars -> secrest in workflow for docker login

* fixed errors in secret names

* changed context for build; added chckout to dev in Dockers

* action up

* action up

* correct path to Dockerfiles in action

* Added psutil reinstall; reworked open3d kill

* Standardized Dockerfiles for better memory handling

* Dockerfiels psutil update

* Dockerfiles update

* Finalized Docerfiles; added arm64

* Finalized Docerfiles; added arm64

* Standardized Dockerfile.vnc

* Fixed deploy.py mistake; mistake in Dockerfile

* Standardaized Dockerfiles

* Comments
added better comments;
added missing restructuredtext comments for function + fix or older ones;
added typing to every function;
updated README

* Updated typing and circular imports

* updated urdf file to get rid of non-uniform axes; added exercise 1,2 readmes

* added scipy to requirements; added readme for exercise 3

* Bugfixes
added check fo -1 in in raybatch which means no contact;
added correct collision mesh for icub sole/foot/boot

* exercise_4 README

* Updated README for exercise 4 so it works also with sphinx

* exercise 5

* Changes for grasper
added timeout to movements;
changed behaviour when joints outside limits are inserted;
visualizer now correctly shows when fixed objects change their position

* updated setup.py; clean up

* Packaging updates
reworked setup.p
added manifest.in and licence
added github action for auto pypi publish

* updated setup.p version; updated dockers

* README up

* pycub folder deletion from docker after installation

File: iCub/full.urdf (robot description, URDF)
Before this commit: robot iCub, 103 links, 102 joints
Links:
- link l_eye_pupil: geometry collision mesh filename=package://iCub/meshes/visual/l_eye_pupil.obj scale=1.0 1.0 1.0; visual mesh filename=package://iCub/meshes/visual/l_eye_pupil.obj scale=1.0 1.0 1.0
- link l_foot: geometry collision mesh filename=package://iCub/meshes/visual/sim_sea_2-5_l_sole_prt-binary.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 scale=0.001 0.001 0.001; visual mesh filename=package://iCub/meshes/visual/sim_sea_2-5_l_sole_prt-binary.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 scale=0.001 0.001 0.001
- link r_eye_pupil: geometry collision mesh filename=package://iCub/meshes/visual/r_eye_pupil.obj scale=1.0 1.0 1.0; visual mesh filename=package://iCub/meshes/visual/r_eye_pupil.obj scale=1.0 1.0 1.0
- link r_foot: geometry collision mesh filename=package://iCub/meshes/visual/sim_sea_2-5_r_sole_prt-binary.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 scale=0.001 0.001 0.001; visual mesh filename=package://iCub/meshes/visual/sim_sea_2-5_r_sole_prt-binary.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 scale=0.001 0.001 0.001
Joints:
- joint l_shoulder_pitch: axis 0.965926 0.0 0.258819 -> 0.9659258492011169 0 0.25881895959357540
- joint l_shoulder_roll: axis -0.258819 2.77555756156e-17 0.965926 -> -0.2588189595935754 0 0.9659258492011169
- joint l_shoulder_yaw: axis 0.965925843882 2.22044604925e-16 0.258818979447 -> 0.9659258492011169 0 0.2588189595935754
- joint l_wrist_pitch: axis 0.258818979447 0.0 -0.965925843882 -> 0.2588189595935754 0.0 -0.9659258492011169
- joint l_wrist_prosup: axis 0.965925843882 2.22044604925e-16 0.258818979447 -> 0.9659258492011169 0 0.2588189595935754
- joint r_shoulder_pitch: axis -0.965925926173 0.0 0.258819275525 -> -0.9659257753743923 0.0 0.25881923511860305
- joint r_shoulder_roll: axis -0.258819 -2.77555756156e-17 -0.965926 -> -0.2588189595935754 0 -0.9659258492011169
- joint r_shoulder_yaw: axis 0.965925843882 -2.22044604925e-16 -0.258818979447 -> 0.9659258492011169 0 -0.2588189595935754
- joint r_wrist_pitch: axis 0.258818979447 0.0 0.965925843882 -> 0.25881895959357540 0 0.9659258492011169
- joint r_wrist_prosup: axis 0.965925843882 -2.22044604925e-16 -0.258818979447 -> 0.9659258492011169 0 -0.2588189595935754
